File: Tarjeta_de_presentacion.kicad_pcb (KiCad board)
At the start: 2 copper layers, 85 x 54 mm, 24 parts, among them J1 Batería, J2 Conn_01x06, J3 Directa, J4 Conn_01x07, J5 Conn_01x09, SW1 Reset, U1 ATMEGA328P-AU, Y1 Crystal

Commit message: //
//
Parts:
- removed C2: C_Small, Capacitors_SMD:C_0805_HandSoldering
- J3: footprint Pin_Headers:Pin_Header_Straight_1x02_Pitch2.54mm -> Librerias_FootPrints:Conector_Directo_SMD
- SW1: footprint Boton_Single -> Librerias_FootPrints:Boton_Single
- moved J2 34.4 mm to (80.0, 47.2), turned to 90 degrees
- moved 1K1 31.1 mm to (77.8, 54.5), turned to 315 degrees
- moved 1K3 27.5 mm to (72.7, 54.8), turned to 315 degrees
- moved C4 26.5 mm to (82.5, 62.5), turned to 135 degrees
- moved D1 25.9 mm to (61.6, 50.7), turned to 315 degrees
- moved 1K4 25.1 mm to (67.8, 55.5), turned to 315 degrees
- moved D4 24.3 mm to (49.6, 50.7), turned to 315 degrees
- moved D3 24.2 mm to (55.6, 50.7), turned to 315 degrees
- moved R1 14.3 mm to (93.9, 55.0), turned to 0 degrees
- moved C1 13.8 mm to (94.0, 51.5)
- moved J3 13.7 mm to (48.3, 85.7)
- moved J4 10.1 mm to (117.2, 46.9)
- moved D2 7.21 mm to (57.3, 88.2), turned to 315 degrees
- moved J1 7.16 mm to (56.2, 69.8)
- moved Y1 6.98 mm to (79.8, 69.5)
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Connections:
- J1 pad 1: /VDD -> /GND
- J1 pad 2: /GND -> /VDD
Routing:
- net /VDD: track 0.00 -> 104.9 mm
- net /A0: track 0.00 -> 43.9 mm
- net /A1: track 0.00 -> 41.3 mm
- net /RESET: track 0.00 -> 35.2 mm
- net /A2: track 0.00 -> 34.8 mm
- net /A3: track 0.00 -> 33.4 mm
- net /TX: track 0.00 -> 33.1 mm
- net /SDA: track 0.00 -> 32.0 mm
- net /SCL: track 0.00 -> 30.6 mm
- net /D4: track 0.00 -> 28.3 mm
- net /RX: track 0.00 -> 27.5 mm
- net /D3: track 0.00 -> 24.0 mm
- net /D5: track 0.00 -> 23.4 mm
- net /D2: track 0.00 -> 23.4 mm
- net /D6: track 0.00 -> 22.0 mm
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
Commit message: //
//
Parts:
- added 1K5: R_Small, Resistors_SMD:R_0805_HandSoldering, F.Cu at (57.6, 45.4)
- added D5: POW_BAT_F, Diodes_SMD:D_0805, B.Cu at (49.0, 45.8)
- moved 1K2 8.54 mm to (55.3, 86.3)
- moved D2 2.83 mm to (59.3, 90.2), turned to 135 degrees
- moved C4 2.02 mm to (81.0, 63.8)
- moved JP1 1.62 mm to (93.6, 81.9)
- moved C5 1.59 mm to (92.1, 83.3)
Connections:
- J2 pad 2: (no net) -> Net-(J2-Pad2)
- U1 pad 19: (no net) -> Net-(U1-Pad19)
- U1 pad 22: (no net) -> Net-(U1-Pad22)
Routing:
- net /GND: track 0.00 -> 469.8 mm, vias 0 -> 31
- net /VDD: track 104.9 -> 213.3 mm
- net Net-(1K2-Pad1): track 8.21 -> 3.19 mm
- added copper zone on B.Cu, net /GND
- added copper zone on F.Cu, net /GND
- added copper zone on F.Cu, net /VDD

Commit message: //
//
Parts:
- added G***: LOGO, Figuras:Informacion_Front_Solder_Mask, B.Cu at (87.0, 71.6)
- added REF**: QFN-32, Housings_DFN_QFN:QFN-32-1EP_5x5mm_Pitch0.5mm, F.Cu at (115.0, 66.0)
- added REF**: R_1210, Resistors_SMD:R_1210, F.Cu at (123.4, 71.6)
- added REF**: BGA-48, SMD_Packages:BGA-48, F.Cu at (110.6, 91.2)
- added REF**: PQFP-44, Housings_QFP:PQFP-44_10x10mm_Pitch0.8mm, F.Cu at (110.2, 78.4)
- added REF**: SOIC-14, Housings_SOIC:SOIC-14_3.9x8.7mm_Pitch1.27mm, F.Cu at (123.0, 89.0)
- added REF**: MSOP-16, Housings_SSOP:MSOP-16_3x4mm_Pitch0.5mm, F.Cu at (123.5, 78.7)
- added REF**: R_0201, Resistors_SMD:R_0201, F.Cu at (123.4, 52.1)
- added REF**: R_0402, Resistors_SMD:R_0402, F.Cu at (123.4, 55.1)
- added REF**: R_0603, Resistors_SMD:R_0603, F.Cu at (123.4, 58.4)
- added REF**: R_0805, Resistors_SMD:R_0805, F.Cu at (123.4, 62.2)
- added REF**: R_1206, Resistors_SMD:R_1206, F.Cu at (123.4, 66.5)
- J2: footprint Pin_Headers:Pin_Header_Straight_1x06_Pitch2.54mm -> Librerias_FootPrints:RS232
- J4: footprint Pin_Headers:Pin_Header_Straight_1x07_Pitch2.54mm -> Librerias_FootPrints:RST_SPI_ANALOG
- J5: footprint Pin_Headers:Pin_Header_Straight_1x09_Pitch2.54mm -> Librerias_FootPrints:D9-D5_SPI
- moved D4 12.9 mm to (62.5, 50.2)
- moved D3 12.5 mm to (68.0, 50.2)
- moved D1 11.8 mm to (73.4, 50.2)
- moved D5 5.99 mm to (52.9, 50.4)
- moved 1K5 4.17 mm to (56.6, 49.5), turned to 135 degrees
Routing:
- net /GND: track 469.8 -> 443.1 mm, vias 31 -> 33
- net Net-(1K4-Pad1): track 17.9 -> 5.15 mm
- net Net-(1K3-Pad1): track 16.4 -> 4.16 mm
- net Net-(1K1-Pad1): track 15.4 -> 3.75 mm
- net Net-(1K5-Pad1): track 0.00 -> 3.60 mm, vias 0 -> 1
- net /VDD: track 213.3 -> 214.5 mm
Other:
- board text added: "+"
- board text added: "-"
- board text added: "FootPrints"
