File: Tarjeta_de_presentacion.sch (KiCad schematic (older format))
At the start: 23 parts, among them J1 Batería, J2 Conn_01x06, J3 Directa, J4 Pines analógicos, J5 Pines Digitales, J6 SPI, J7 I2C, J8 Fuente, SW1 Reset, U1 ATMEGA328P-AU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

Commit message: /
//
Parts:
- removed J4: Pines analógicos, Pin_Headers:Pin_Header_Straight_1x06_Pitch2.54mm, symbol Conn_01x06
- removed J5: Pines Digitales, Pin_Headers:Pin_Header_Straight_1x08_Pitch2.54mm, symbol Conn_01x08
- removed J6: SPI, Pin_Headers:Pin_Header_Straight_1x04_Pitch2.54mm, symbol Conn_01x04
- removed J7: I2C, Pin_Headers:Pin_Header_Straight_1x02_Pitch2.54mm, symbol Conn_01x02
- removed J8: Fuente, Pin_Headers:Pin_Header_Straight_1x04_Pitch2.54mm, symbol Conn_01x04
- added 1K3, 1K4: R_Small, Resistors_SMD:R_0805_HandSoldering, symbol R_Small
- added D3: Test_D3, Diodes_SMD:D_0805, symbol D_Small
- added D4: Test_D4, Diodes_SMD:D_0805, symbol D_Small
- added J4: Conn_01x07, Pin_Headers:Pin_Header_Straight_1x07_Pitch2.54mm, symbol Conn_01x07
- added J5: Conn_01x09, Pin_Headers:Pin_Header_Straight_1x09_Pitch2.54mm, symbol Conn_01x09
- D1: value D_Small -> Test_D2
- D2: value D_Small -> POW
- J1: footprint Pin_Headers:Pin_Header_Straight_1x02_Pitch2.54mm -> Librerias_FootPrints:Holder_Battery
- SW1: footprint (none) -> Librerias_FootPrints:Boton_Single
- Y1: footprint (none) -> Crystals:Crystal_HC49-4H_Vertical
Connections:
- net A0: now also J4.1 (Pin_1)
- net A1: now also J4.2 (Pin_2)
- net A2: now also J4.3 (Pin_3)
- net A3: now also J4.4 (Pin_4)
- net D3: now also 1K3.2
- net D4: now also 1K4.2
- net D5: now also J5.9 (Pin_9)
- net D6: now also J5.8 (Pin_8)
- net D7: now also J5.7 (Pin_7)
- net D8: now also J5.6 (Pin_6)
- net D9: now also J5.5 (Pin_5)
- net GND: now also D3.1 (K), D4.1 (K)
- net MISO: now also J5.2 (Pin_2)
- net MOSI: now also J5.3 (Pin_3)
- net RESET: now also J4.7 (Pin_7)
- net SCK: now also J5.1 (Pin_1)
- net SCL: now also J4.6 (Pin_6)
- net SDA: now also J4.5 (Pin_5)
- net SS: now also J5.4 (Pin_4)
- net A6: no longer names the net of U1.19 (ADC6)
- net A7: no longer names the net of U1.22 (ADC7)
- new net: 1K3.1, D3.2 (A)
- new net: 1K4.1, D4.2 (A)
- no-connect marks 1 -> 3
Other:
- note added: "LED DE ALIMENTACIÓN"
- note added: "LEDS DE PRUEBA"
- note removed: "*Recodar A6-A7\nNetamente analógicos"
- note removed: "COMUNICACIÓN I2C Y SPI"
- note removed: "LED DE PRUEBA"
- note removed: "OTROS"
- moved on the sheet: 1K1, 1K2, D1, D2

Commit message: //
//
Parts:
- removed C2: C_Small, Capacitors_SMD:C_0805_HandSoldering, symbol C_Small
- J3: footprint Pin_Headers:Pin_Header_Straight_1x02_Pitch2.54mm -> Librerias_FootPrints:Conector_Directo_SMD
Connections:
- net GND: now also J1.1 (Pin_1); no longer J1.2 (Pin_2)
- net VDD: now also J1.2 (Pin_2); no longer J1.1 (Pin_1)
Other:
- moved on the sheet: C4, C5
Changed lines of the file:
@@
 F 0 "J3" H 1950 1250 50  0000 C CNN
 F 1 "Directa" H 1950 950 50  0000 C CNN
-F 2 "Pin_Headers:Pin_Header_Straight_1x02_Pitch2.54mm" H 1950 1150 50  0001 C CNN
+F 2 "Librerias_FootPrints:Conector_Directo_SMD" H 1950 1150 50  0001 C CNN
 F 3 "" H 1950 1150 50  0001 C CNN
 	1    1950 1150
@@
 Wire Wire Line
 	1100 1350 1100 1650
+Text Label 1100 1650 1    60   ~ 0
+VDD
 Text Label 1000 1650 1    60   ~ 0
-VDD
-Text Label 1100 1650 1    60   ~ 0
 GND
 Wire Wire Line
@@
 U 1 1 5B0AE8AB
 P 10100 2450
-F 0 "1K1" H 10130 2470 50  0000 L CNN
+F 0 "1K1" H 10130 2470 50  0001 L CNN
 F 1 "R_Small" H 10130 2410 50  0001 L CNN
 F 2 "Resistors_SMD:R_0805_HandSoldering" H 10100 2450 50  0001 C CNN
@@
 CAPACITORES DESACOPLE
 $Comp
-L C_Small C2
-U 1 1 5B0AF08B
+L C_Small C4
+U 1 1 5B0AF154
 P 1100 5900
-F 0 "C2" H 1110 5970 50  0000 L CNN
+F 0 "C4" H 1110 5970 50  0000 L CNN
 F 1 "C_Small" H 1110 5820 50  0001 L CNN
 F 2 "Capacitors_SMD:C_0805_HandSoldering" H 1100 5900 50  0001 C CNN
@@
 $EndComp
 $Comp
-L C_Small C4
-U 1 1 5B0AF154
+L C_Small C5
+U 1 1 5B0AF17F
 P 1350 5900
-F 0 "C4" H 1360 5970 50  0000 L CNN
+F 0 "C5" H 1360 5970 50  0000 L CNN
 F 1 "C_Small" H 1360 5820 50  0001 L CNN
 F 2 "Capacitors_SMD:C_0805_HandSoldering" H 1350 5900 50  0001 C CNN
@@
 	1    0    0    -1
 $EndComp
-$Comp
-L C_Small C5
-U 1 1 5B0AF17F
-P 1600 5900
-F 0 "C5" H 1610 5970 50  0000 L CNN
-F 1 "C_Small" H 1610 5820 50  0001 L CNN
-F 2 "Capacitors_SMD:C_0805_HandSoldering" H 1600 5900 50  0001 C CNN
-F 3 "" H 1600 5900 50  0001 C CNN
-	1    1600 5900
-	1    0    0    -1
-$EndComp
+Wire Wire Line
+	1350 5650 1350 5800
 Wire Wire Line
 	1100 5800 1100 5650
 Wire Wire Line
-	1100 5650 1600 5650
-Wire Wire Line
-	1600 5650 1600 5800
-Wire Wire Line
-	1350 5800 1350 5650
-Connection ~ 1350 5650
-Wire Wire Line
-	1600 6000 1600 6200
-Wire Wire Line
-	1600 6200 1100 6200
-Wire Wire Line
-	1100 6200 1100 6000
-Wire Wire Line
 	1350 6000 1350 6200
-Connection ~ 1350 6200
-Text Label 1150 5650 0    60   ~ 0
-VDD
-Text Label 1150 6200 0    60   ~ 0
+Wire Wire Line
+	1100 6000 1100 6200
+Text Label 1200 5650 0    60   ~ 0
+VDD
+Text Label 1200 6200 0    60   ~ 0
 GND
 Wire Notes Line
@@
 Wire Wire Line
 	3450 1900 3150 1900
-Text Label 3150 1900 0    60   ~ 0
-VDD
 Text Label 3300 3400 0    60   ~ 0
 GND
@@
 U 1 1 5B0DFA8F
 P 10100 2800
-F 0 "1K3" H 10130 2820 50  0000 L CNN
+F 0 "1K3" H 10130 2820 50  0001 L CNN
 F 1 "R_Small" H 10130 2760 50  0001 L CNN
 F 2 "Resistors_SMD:R_0805_HandSoldering" H 10100 2800 50  0001 C CNN
@@
 U 1 1 5B0DFAE4
 P 10100 3100
-F 0 "1K4" H 10130 3120 50  0000 L CNN
+F 0 "1K4" H 10130 3120 50  0001 L CNN
 F 1 "R_Small" H 10130 3060 50  0001 L CNN
 F 2 "Resistors_SMD:R_0805_HandSoldering" H 10100 3100 50  0001 C CNN
@@
 Text Label 8700 1650 1    60   ~ 0
 RESET
+Text Label 3150 1900 0    60   ~ 0
+VDD
+Wire Wire Line
+	1100 5650 1350 5650
+Wire Wire Line
+	1100 6200 1350 6200
 $EndSCHEMATC

Commit message: //
//
Parts:
- added 1K5: R_Small, Resistors_SMD:R_0805_HandSoldering, symbol R_Small
- added D5: POW_BAT_F, Diodes_SMD:D_0805, symbol D_Small
Connections:
- net GND: now also D5.1 (K)
- net VDD: now also 1K5.2
- new net: 1K5.1, D5.2 (A)
Changed lines of the file:
@@
 Wire Wire Line
 	1100 6200 1350 6200
+$Comp
+L D_Small D5
+U 1 1 5B137531
+P 10400 3350
+F 0 "D5" H 10350 3430 50  0000 L CNN
+F 1 "POW_BAT_F" H 10250 3270 50  0000 L CNN
+F 2 "Diodes_SMD:D_0805" V 10400 3350 50  0001 C CNN
+F 3 "" V 10400 3350 50  0001 C CNN
+	1    10400 3350
+	-1   0    0    1
+$EndComp
+Wire Wire Line
+	10500 3350 10800 3350
+Text Label 10800 3350 2    60   ~ 0
+GND
+$Comp
+L R_Small 1K5
+U 1 1 5B137D3F
+P 10100 3350
+F 0 "1K5" H 10130 3370 50  0001 L CNN
+F 1 "R_Small" H 10130 3310 50  0001 L CNN
+F 2 "Resistors_SMD:R_0805_HandSoldering" H 10100 3350 50  0001 C CNN
+F 3 "" H 10100 3350 50  0001 C CNN
+	1    10100 3350
+	0    1    1    0
+$EndComp
+Wire Wire Line
+	10300 3350 10200 3350
+Wire Wire Line
+	10000 3350 9750 3350
+Text Label 9750 3350 0    60   ~ 0
+VDD
 $EndSCHEMATC

Commit message: //
//
Parts:
- J2: footprint Pin_Headers:Pin_Header_Straight_1x06_Pitch2.54mm -> Librerias_FootPrints:RS232
- J4: footprint Pin_Headers:Pin_Header_Straight_1x07_Pitch2.54mm -> Librerias_FootPrints:RST_SPI_ANALOG
- J5: footprint Pin_Headers:Pin_Header_Straight_1x09_Pitch2.54mm -> Librerias_FootPrints:D9-D5_SPI
Changed lines of the file:
@@
 F 0 "J2" H 8600 2550 50  0000 C CNN
 F 1 "Conn_01x06" H 8600 1850 50  0001 C CNN
-F 2 "Pin_Headers:Pin_Header_Straight_1x06_Pitch2.54mm" H 8600 2250 50  0001 C CNN
+F 2 "Librerias_FootPrints:RS232" H 8600 2250 50  0001 C CNN
 F 3 "" H 8600 2250 50  0001 C CNN
 	1    8600 2250
@@
 F 0 "J5" H 9650 1650 50  0000 C CNN
 F 1 "Conn_01x09" H 9650 650 50  0000 C CNN
-F 2 "Pin_Headers:Pin_Header_Straight_1x09_Pitch2.54mm" H 9650 1150 50  0001 C CNN
+F 2 "Librerias_FootPrints:D9-D5_SPI" H 9650 1150 50  0001 C CNN
 F 3 "" H 9650 1150 50  0001 C CNN
 	1    9650 1150
@@
 F 0 "J4" H 8400 1550 50  0000 C CNN
 F 1 "Conn_01x07" H 8400 750 50  0000 C CNN
-F 2 "Pin_Headers:Pin_Header_Straight_1x07_Pitch2.54mm" H 8400 1150 50  0001 C CNN
+F 2 "Librerias_FootPrints:RST_SPI_ANALOG" H 8400 1150 50  0001 C CNN
 F 3 "" H 8400 1150 50  0001 C CNN
 	1    8400 1150
